File: projects/PCB_New/capstoneSchematic.brd (EAGLE design)
At the start: 70.2 x 66.2 mm, 55 parts, among them J1 10118192-0001LF, J2 FTSH-107-01-L-DV-K-A, U1 STM32L476VCT6, U2 LD39050PU33R, U3 74LVC125APW,118, Y1 ABLS-8.000MHZ-B2-T, Y2 ECS-.327-12.5-12QS-TR

Commit message: fixes
Parts:
- moved C11 3.43 mm to (36.6, 47.2)
- moved C1 1.67 mm to (19.8, 32.0)
- moved R15 1.40 mm to (62.7, 46.7)
- moved R3 0.38 mm to (28.4, 43.3)
- moved U$1 0.13 mm to (27.1, 61.0)
Routing:
- net SWDIO: track 64.9 -> 99.2 mm, vias 0 -> 2
- net NRST: track 120.1 -> 131.5 mm, vias 0 -> 2
- net SWCLK: track 124.6 -> 128.5 mm, vias 4 -> 7
- net SWO: track 69.7 -> 67.0 mm
- net 5V_IN: track 66.8 -> 64.7 mm
- net GND: track 104.7 -> 106.7 mm
- net N$10: track 2.59 -> 3.85 mm
- net N$12: track 16.7 -> 15.5 mm
- net 5V: track 131.3 -> 132.1 mm
- net 3V3: track 72.8 -> 72.2 mm
- net N$25: track 4.32 -> 3.76 mm

Commit message: V2 Changes
Parts:
- removed J2: FTSH-107-01-L-DV-K-A, ce-capstone:FTSH10701LDVKA
- added J5: (no value), SparkFun-Connectors:2X8
- moved R10 17.1 mm to (53.2, 31.9)
- moved R14 17.1 mm to (50.5, 31.9)
- moved R16 17.1 mm to (67.8, 29.6)
- moved U3 17.1 mm to (59.8, 34.4)
- moved R15 17.1 mm to (64.0, 29.7)
- moved DAC4 7.81 mm to (24.1, 15.1)
- moved USART2 6.48 mm to (28.4, 7.49)
- moved U2 0.89 mm to (32.6, 7.49)
- moved SPI1 0.28 mm to (40.9, 8.00)
Connections:
- net 5V: now also J5.3; no longer J2.3
- net GND: now also J5.11, J5.5, J5.7; no longer J2.11, J2.5, J2.7
- net NRST: now also J5.12; no longer J2.12
- net SWCLK: now also J5.6, J5.9; no longer J2.6, J2.9
- net SWDIO: now also J5.4; no longer J2.4
- net SWO: now also J5.8; no longer J2.8
- net USART_RX: now also J5.13; no longer J2.13
- net USART_TX: now also J5.14; no longer J2.14
Routing:
- net NRST: track 131.5 -> 102.1 mm
- net CS_LLS: track 44.0 -> 26.5 mm
- net DI_LLS: track 41.6 -> 24.6 mm
- net D0_LLS: track 48.3 -> 31.8 mm
- net MOSI: track 26.0 -> 12.1 mm
- net SCK: track 29.1 -> 15.7 mm
- net SCK_LLS: track 42.0 -> 28.7 mm
- net CS: track 37.6 -> 26.6 mm
- net SWCLK: track 128.5 -> 136.7 mm
- net N$15: track 19.2 -> 11.5 mm, vias 2 -> 0
- net MISO: track 40.7 -> 34.4 mm
- net SWDIO: track 99.2 -> 104.3 mm
- net USART_RX: track 106.6 -> 101.6 mm
- net N$23: track 19.4 -> 23.3 mm
- net N$22: track 22.6 -> 26.3 mm
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Other:
- board text added: "Smart Home Assistant PCB V2"
- board text removed: "Smart Home Assistant PCB V1"

Commit message: SD Changes
Connections:
- net CS: now also R10.1; no longer R15.1
- net SCK: now also R15.1; no longer R10.1
Routing:
- net SCK: track 15.7 -> 25.9 mm
- net CS: track 26.6 -> 17.9 mm
Changed lines of the file:
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@@
 <wire x1="41.332" y1="27.489" x2="39.631" y2="27.489" width="0.2032" layer="1"/>
 <wire x1="41.332" y1="27.489" x2="41.529" y2="27.686" width="0.2032" layer="1"/>
-<contactref element="R10" pad="1"/>
 <wire x1="41.529" y1="27.686" x2="41.529" y2="28.575" width="0.2032" layer="16"/>
-<wire x1="50.419" y1="29.464" x2="42.4273125" y2="29.464" width="0.2032" layer="16"/>
-<wire x1="50.419" y1="29.464" x2="50.673" y2="29.718" width="0.2032" layer="16"/>
-<via x="50.673" y="29.718" extent="1-16" drill="0.35"/>
-<wire x1="50.673" y1="29.718" x2="51.704" y2="29.718" width="0.2032" layer="1"/>
-<wire x1="51.704" y1="29.718" x2="53.213" y2="31.227" width="0.2032" layer="1"/>
+<wire x1="42.4273125" y1="29.464" x2="50.419" y2="29.464" width="0.2032" layer="16"/>
 <wire x1="41.529" y1="28.575" x2="42.4273125" y2="29.4733125" width="0.2032" layer="16"/>
 <wire x1="42.4273125" y1="29.4733125" x2="42.4273125" y2="29.464" width="0.2032" layer="16"/>
+<contactref element="R15" pad="1"/>
+<wire x1="50.419" y1="29.464" x2="62.3866" y2="29.464" width="0.2032" layer="16"/>
+<wire x1="62.3866" y1="29.464" x2="62.7676" y2="29.083" width="0.2032" layer="16"/>
+<via x="62.7676" y="29.083" extent="1-16" drill="0.35"/>
+<wire x1="62.7676" y1="29.083" x2="63.993" y2="29.083" width="0.2032" layer="1"/>
+<wire x1="63.993" y1="29.083" x2="64.008" y2="29.068" width="0.1524" layer="1"/>
 </signal>
 <signal name="D0_LLS">
@@
 <signal name="SCK_LLS">
 <contactref element="U3" pad="8"/>
-<wire x1="62.742" y1="32.367" x2="62.742" y2="27.436" width="0.2032" layer="1"/>
-<wire x1="59.69" y1="24.384" x2="62.742" y2="27.436" width="0.2032" layer="1"/>
+<wire x1="62.742" y1="32.367" x2="62.742" y2="31.732" width="0.2032" layer="1"/>
+<wire x1="62.742" y1="31.732" x2="61.218" y2="30.208" width="0.2032" layer="1"/>
+<wire x1="61.218" y1="30.208" x2="61.218" y2="25.912" width="0.2032" layer="1"/>
+<wire x1="59.69" y1="24.384" x2="61.218" y2="25.912" width="0.2032" layer="1"/>
 <via x="59.69" y="24.384" extent="1-16" drill="0.35"/>
 <contactref element="U$2" pad="P$5"/>
@@
 <wire x1="42.322" y1="27.02" x2="42.418" y2="26.924" width="0.2032" layer="1"/>
 <via x="42.418" y="26.924" extent="1-16" drill="0.35"/>
-<wire x1="42.418" y1="26.924" x2="46.99" y2="26.924" width="0.2032" layer="16"/>
-<contactref element="R15" pad="1"/>
-<wire x1="46.99" y1="26.924" x2="64.008" y2="26.924" width="0.2032" layer="16"/>
-<via x="64.008" y="26.924" extent="1-16" drill="0.35"/>
-<wire x1="64.008" y1="26.924" x2="64.008" y2="29.068" width="0.2032" layer="1"/>
+<wire x1="42.418" y1="26.924" x2="53.086" y2="26.924" width="0.2032" layer="16"/>
+<via x="53.086" y="26.924" extent="1-16" drill="0.35"/>
+<contactref element="R10" pad="1"/>
+<wire x1="53.086" y1="26.924" x2="53.213" y2="27.051" width="0.2032" layer="1"/>
+<wire x1="53.213" y1="27.051" x2="53.213" y2="31.227" width="0.2032" layer="1"/>
 </signal>
 <signal name="N$9">

Commit message: SD Buffer Changes
Parts:
- removed R10, R14, R15, R16: RC0402FR-073K3L, RC0402FR-073K3L:RESC1005X40
- removed U3: 74LVC125APW,118, 74LVC125APW_118:IC_74LVC125APW,118
Connections:
- removed net CS_LLS: U$2.P$2, U3.6
- removed net D0_LLS: R16.1, U$2.P$7
- removed net DI_LLS: U$2.P$3, U3.3
- removed net N$13: R14.2, U3.2
- removed net N$24: R10.2, U3.5
- removed net N$25: R15.2, U3.9
- removed net N$26: R16.2, U3.12
- removed net SCK_LLS: U$2.P$5, U3.8
- net 3V3: no longer U3.14
- net CS: now also U$2.P$2; no longer R10.1
- net GND: no longer U3.1, U3.10, U3.13, U3.4, U3.7
- net MISO: now also U$2.P$7; no longer U3.11
- net MOSI: now also U$2.P$3; no longer R14.1
- net SCK: now also U$2.P$5; no longer R15.1
Routing:
- net D0_LLS: track 31.8 -> 0.00 mm
- net SCK_LLS: track 28.7 -> 0.00 mm, vias 2 -> 0
- net CS_LLS: track 26.5 -> 0.00 mm, vias 2 -> 0
- net DI_LLS: track 24.6 -> 0.00 mm
- net MOSI: track 12.1 -> 33.1 mm
- net CS: track 17.9 -> 29.1 mm
- net GND: track 105.8 -> 94.9 mm, vias 53 -> 48
- net N$13: track 8.92 -> 0.00 mm
- net N$26: track 7.81 -> 0.00 mm
- net MISO: track 34.4 -> 29.6 mm
- net N$24: track 4.19 -> 0.00 mm
- net N$25: track 3.76 -> 0.00 mm
- net SCK: track 25.9 -> 29.4 mm
- net 3V3: track 72.2 -> 70.4 mm, vias 22 -> 21

Commit message: Final Fix
Connections:
- net N$11 renamed USART3_RX
- net N$14 renamed USART4_TX
- net N$16 renamed USART4_RX
- net N$17 renamed SPI1_SCK
- net N$18 renamed SPI1_MISO
- net N$19 renamed USART1_RX
- net N$20 renamed USART1_TX
- net N$22 renamed USART2_TX
- net N$23 renamed USART2_RX
- net N$9 renamed USART3_TX
- net 3V3: now also J5.10
Routing:
- net 3V3: track 70.4 -> 72.5 mm, vias 21 -> 22
Changed lines of the file:
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@@
 <wire x1="35.814" y1="49.403" x2="31.369" y2="53.848" width="0.2032" layer="16"/>
 <wire x1="35.306" y1="47.117" x2="35.306" y2="48.895" width="0.2032" layer="1"/>
+<contactref element="J5" pad="10"/>
+<wire x1="14.605" y1="8.636" x2="14.605" y2="10.795" width="0.2032" layer="1"/>
+<via x="14.605" y="10.795" extent="1-16" drill="0.35"/>
 </signal>
 <signal name="N$5">
@@
 <wire x1="58.42" y1="15.113" x2="58.42" y2="11.811" width="0.2032" layer="1"/>
 </signal>
-<signal name="N$9">
+<signal name="USART3_TX">
 <contactref element="U1" pad="33"/>
 <contactref element="USART3" pad="2"/>
@@
 <wire x1="48.768" y1="21.463" x2="50.038" y2="20.193" width="0.2032" layer="1"/>
 </signal>
-<signal name="N$11">
+<signal name="USART3_RX">
 <contactref element="U1" pad="34"/>
 <contactref element="USART3" pad="1"/>
@@
 <wire x1="29.75" y1="25.17" x2="29.75" y2="23.7452125" width="0.2032" layer="1"/>
 </signal>
-<signal name="N$14">
+<signal name="USART4_TX">
 <contactref element="U1" pad="78"/>
 <contactref element="USART4" pad="2"/>
@@
 <wire x1="35.306" y1="44.95293125" x2="35.306" y2="43.434" width="0.2032" layer="16"/>
 </signal>
-<signal name="N$16">
+<signal name="USART4_RX">
 <contactref element="U1" pad="79"/>
 <contactref element="USART4" pad="1"/>
@@
 <wire x1="27.051" y1="50.165" x2="27.051" y2="51.943" width="0.2032" layer="1"/>
 </signal>
-<signal name="N$19">
+<signal name="USART1_RX">
 <contactref element="U1" pad="69"/>
 <contactref element="USART1" pad="1"/>
@@
 <wire x1="49.276" y1="40.64" x2="49.276" y2="38.481" width="0.2032" layer="1"/>
 </signal>
-<signal name="N$20">
+<signal name="USART1_TX">
 <contactref element="U1" pad="68"/>
 <contactref element="USART1" pad="2"/>
@@
 <wire x1="48.006" y1="37.211" x2="49.276" y2="35.941" width="0.2032" layer="1"/>
 </signal>
-<signal name="N$22">
+<signal name="USART2_TX">
 <contactref element="U1" pad="25"/>
 <contactref element="USART2" pad="2"/>
@@
 <wire x1="25.908" y1="9.271" x2="25.908" y2="7.493" width="0.2032" layer="1"/>
 </signal>
-<signal name="N$23">
+<signal name="USART2_RX">
 <contactref element="U1" pad="26"/>
 <contactref element="USART2" pad="1"/>
@@
 <wire x1="27.4292" y1="18.4122" x2="24.13" y2="15.113" width="0.2032" layer="1"/>
 </signal>
-<signal name="N$17">
+<signal name="SPI1_SCK">
 <contactref element="U1" pad="30"/>
 <contactref element="SPI1" pad="2"/>
@@
 <wire x1="37.7825" y1="8.5725" x2="38.354" y2="8.001" width="0.2032" layer="1"/>
 </signal>
-<signal name="N$18">
+<signal name="SPI1_MISO">
 <contactref element="U1" pad="31"/>
 <contactref element="SPI1" pad="1"/>

Commit message: Iteration 2 commit
Parts:
- added J2: (no value), SparkFun-Connectors:1X05_LOCK
- added J4: (no value), SparkFun-Connectors:1X02
- moved USART3 35.5 mm to (51.6, 53.1), turned to 180 degrees
- moved C8 5.17 mm to (40.4, 19.7)
- moved D1 3.59 mm to (33.8, 19.8)
- moved D2 3.59 mm to (35.8, 19.8)
- moved R1 3.59 mm to (33.8, 22.2)
- moved R2 3.59 mm to (35.8, 22.2)
- moved C12 1.97 mm to (41.0, 22.5)
Connections:
- new net DFSDM1_CKOUT: J2.4, U1.17
- new net DFSDM1_DATIN0: J2.2, U1.36
- new net GPIO_CS: J4.1, U1.35
- new net SPI1_MOSI: J4.2, U1.32
- net 3V3: now also J2.3
- net GND: now also DAC4.2, J2.1, J2.5
Routing:
- net DFSDM1_CKOUT: track 0.00 -> 79.8 mm, vias 0 -> 4
- net DFSDM1_DATIN0: track 0.00 -> 49.6 mm, vias 0 -> 2
- net USART3_RX: track 28.0 -> 61.6 mm
- net USART3_TX: track 23.9 -> 51.7 mm
- net GPIO_CS: track 0.00 -> 19.2 mm, vias 0 -> 2
- net SPI1_MOSI: track 0.00 -> 13.4 mm
- net N$1: track 2.01 -> 5.33 mm
- net GND: track 94.9 -> 98.1 mm, vias 48 -> 50
- net 3V3: track 72.5 -> 74.5 mm, vias 22 -> 23
- net N$2: track 2.80 -> 4.23 mm
- net USART_TX: track 90.3 -> 89.5 mm
- net SWDIO: track 104.3 -> 104.8 mm
