File: projects/PCB_New/capstoneSchematic.sch (EAGLE design)
At the start: 55 parts, among them J1 10118192-0001LF, J2 FTSH-107-01-L-DV-K-A, U1 STM32L476VCT6, U2 LD39050PU33R, U3 74LVC125APW,118, Y1 ABLS-8.000MHZ-B2-T, Y2 ECS-.327-12.5-12QS-TR

Commit message: V2 Changes
Parts:
- removed J2: FTSH-107-01-L-DV-K-A, ce-capstone:FTSH-107-01-L-DV-K-A
- added J5: (no value), SparkFun-Connectors:CONN_08X2_HEADER
Connections:
- net 5V: now also J5.3; no longer J2.3
- net GND: now also J5.11, J5.5, J5.7; no longer J2.11, J2.5, J2.7
- net NRST: now also J5.12; no longer J2.12
- net SWCLK: now also J5.6, J5.9; no longer J2.6, J2.9
- net SWDIO: now also J5.4; no longer J2.4
- net SWO: now also J5.8; no longer J2.8
- net USART_RX: now also J5.13; no longer J2.13
- net USART_TX: now also J5.14; no longer J2.14
Other:
- moved on the sheet: R10, R14, R15, R16, U$2, U3

Commit message: SD Changes
Connections:
- net CS: now also R10.1; no longer R15.1
- net SCK: now also R15.1; no longer R10.1
Changed lines of the file:
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@@
 </segment>
 <segment>
-<pinref part="R10" gate="G$1" pin="1"/>
-<wire x1="170.18" y1="83.82" x2="165.1" y2="83.82" width="0.1524" layer="91"/>
-<label x="165.1" y="83.82" size="1.778" layer="95"/>
+<pinref part="R15" gate="G$1" pin="1"/>
+<wire x1="170.18" y1="76.2" x2="165.1" y2="76.2" width="0.1524" layer="91"/>
+<label x="165.1" y="76.2" size="1.778" layer="95"/>
 </segment>
 </net>
@@
 </segment>
 <segment>
-<pinref part="R15" gate="G$1" pin="1"/>
-<wire x1="170.18" y1="76.2" x2="165.1" y2="76.2" width="0.1524" layer="91"/>
-<label x="165.1" y="76.2" size="1.778" layer="95"/>
+<pinref part="R10" gate="G$1" pin="1"/>
+<wire x1="170.18" y1="83.82" x2="165.1" y2="83.82" width="0.1524" layer="91"/>
+<label x="165.1" y="83.82" size="1.778" layer="95"/>
 </segment>
 </net>

Commit message: SD Buffer Changes
Parts:
- removed R10, R14, R15, R16: RC0402FR-073K3L, RC0402FR-073K3L:RC0402FR-073K3L
- removed U3: 74LVC125APW,118, 74LVC125APW_118:74LVC125APW,118
Connections:
- removed net CS_LLS: U$2.CD_DAT3_CS, U3.2Y
- removed net D0_LLS: R16.1, U$2.DAT0_DO
- removed net DI_LLS: U$2.CMD_DIN, U3.1Y
- removed net N$13: R14.2, U3.1A
- removed net N$24: R10.2, U3.2A
- removed net N$25: R15.2, U3.3A
- removed net N$26: R16.2, U3.4A
- removed net SCK_LLS: U$2.CLK, U3.3Y
- net 3V3: no longer U3.VCC
- net CS: now also U$2.CD_DAT3_CS; no longer R10.1
- net GND: no longer U3.1!OE, U3.2!OE, U3.3!OE, U3.4!OE, U3.GND
- net MISO: now also U$2.DAT0_DO; no longer U3.4Y
- net MOSI: now also U$2.CMD_DIN; no longer R14.1
- net SCK: now also U$2.CLK; no longer R15.1
Other:
- moved on the sheet: C17, C18, C19, C2, C20, C21, C3, C4, C5, D3, J5, R6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

Commit message: Final Fix
Connections:
- net N$11 renamed USART3_RX
- net N$14 renamed USART4_TX
- net N$16 renamed USART4_RX
- net N$17 renamed SPI1_SCK
- net N$18 renamed SPI1_MISO
- net N$19 renamed USART1_RX
- net N$20 renamed USART1_TX
- net N$22 renamed USART2_TX
- net N$23 renamed USART2_RX
- net N$9 renamed USART3_TX
- net 3V3: now also J5.10
Other:
- moved on the sheet: USART1, USART4
Changed lines of the file:
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@@
 <attribute name="NAME" x="47.752" y="-50.8" size="1.778" layer="95" font="vector" rot="R90"/>
 </instance>
-<instance part="USART4" gate="J1" x="86.36" y="116.84" smashed="yes" rot="R270">
-<attribute name="VALUE" x="81.534" y="119.38" size="1.778" layer="96" font="vector" rot="R270"/>
-<attribute name="NAME" x="91.948" y="119.38" size="1.778" layer="95" font="vector" rot="R270"/>
-</instance>
-<instance part="USART1" gate="J1" x="134.62" y="58.42" smashed="yes" rot="R180">
-<attribute name="VALUE" x="137.16" y="63.246" size="1.778" layer="96" font="vector" rot="R180"/>
-<attribute name="NAME" x="137.16" y="52.832" size="1.778" layer="95" font="vector" rot="R180"/>
+<instance part="USART4" gate="J1" x="86.36" y="121.92" smashed="yes" rot="R270">
+<attribute name="VALUE" x="81.534" y="124.46" size="1.778" layer="96" font="vector" rot="R270"/>
+<attribute name="NAME" x="91.948" y="124.46" size="1.778" layer="95" font="vector" rot="R270"/>
+</instance>
+<instance part="USART1" gate="J1" x="142.24" y="58.42" smashed="yes" rot="R180">
+<attribute name="VALUE" x="144.78" y="63.246" size="1.778" layer="96" font="vector" rot="R180"/>
+<attribute name="NAME" x="144.78" y="52.832" size="1.778" layer="95" font="vector" rot="R180"/>
 </instance>
 <instance part="USART2" gate="J1" x="-7.62" y="-15.24" smashed="yes">
@@
 <pinref part="U$2" gate="G$1" pin="VDD"/>
 </segment>
+<segment>
+<pinref part="J5" gate="J1" pin="10"/>
+<wire x1="147.32" y1="149.86" x2="157.48" y2="149.86" width="0.1524" layer="91"/>
+<label x="149.86" y="149.86" size="1.778" layer="95"/>
+</segment>
 </net>
 <net name="N$5" class="0">
@@
 </segment>
 </net>
-<net name="N$9" class="0">
+<net name="USART3_TX" class="0">
 <segment>
 <pinref part="U1" gate="G$1" pin="PC4"/>
 <pinref part="USART3" gate="J1" pin="2"/>
 <wire x1="50.8" y1="-10.16" x2="50.8" y2="-40.64" width="0.1524" layer="91"/>
-</segment>
-</net>
-<net name="N$11" class="0">
+<label x="50.8" y="-35.56" size="1.778" layer="95" rot="R90"/>
+</segment>
+</net>
+<net name="USART3_RX" class="0">
 <segment>
 <pinref part="U1" gate="G$1" pin="PC5"/>
 <pinref part="USART3" gate="J1" pin="1"/>
 <wire x1="53.34" y1="-10.16" x2="53.34" y2="-40.64" width="0.1524" layer="91"/>
-</segment>
-</net>
-<net name="N$14" class="0">
+<label x="53.34" y="-35.56" size="1.778" layer="95" rot="R90"/>
+</segment>
+</net>
+<net name="USART4_TX" class="0">
 <segment>
 <pinref part="U1" gate="G$1" pin="PC10"/>
 <pinref part="USART4" gate="J1" pin="2"/>
-<wire x1="88.9" y1="96.52" x2="88.9" y2="109.22" width="0.1524" layer="91"/>
-</segment>
-</net>
-<net name="N$16" class="0">
+<wire x1="88.9" y1="96.52" x2="88.9" y2="114.3" width="0.1524" layer="91"/>
+<label x="88.9" y="99.06" size="1.778" layer="95" rot="R90"/>
+</segment>
+</net>
+<net name="USART4_RX" class="0">
 <segment>
 <pinref part="U1" gate="G$1" pin="PC11"/>
 <pinref part="USART4" gate="J1" pin="1"/>
-<wire x1="86.36" y1="96.52" x2="86.36" y2="109.22" width="0.1524" layer="91"/>
-</segment>
-</net>
-<net name="N$19" class="0">
+<wire x1="86.36" y1="96.52" x2="86.36" y2="114.3" width="0.1524" layer="91"/>
+<label x="86.36" y="99.06" size="1.778" layer="95" rot="R90"/>
+</segment>
+</net>
+<net name="USART1_RX" class="0">
 <segment>
 <pinref part="U1" gate="G$1" pin="PA10"/>
 <pinref part="USART1" gate="J1" pin="1"/>
-<wire x1="116.84" y1="58.42" x2="127" y2="58.42" width="0.1524" layer="91"/>
-</segment>
-</net>
-<net name="N$20" class="0">
+<wire x1="116.84" y1="58.42" x2="134.62" y2="58.42" width="0.1524" layer="91"/>
+<label x="119.38" y="58.42" size="1.778" layer="95"/>
+</segment>
+</net>
+<net name="USART1_TX" class="0">
 <segment>
 <pinref part="U1" gate="G$1" pin="PA9"/>
 <pinref part="USART1" gate="J1" pin="2"/>
-<wire x1="116.84" y1="55.88" x2="127" y2="55.88" width="0.1524" layer="91"/>
-</segment>
-</net>
-<net name="N$22" class="0">
+<wire x1="116.84" y1="55.88" x2="134.62" y2="55.88" width="0.1524" layer="91"/>
+<label x="119.38" y="55.88" size="1.778" layer="95"/>
+</segment>
+</net>
+<net name="USART2_TX" class="0">
 <segment>
 <pinref part="U1" gate="G$1" pin="PA2"/>
@@
 <wire x1="10.16" y1="12.7" x2="10.16" y2="-12.7" width="0.1524" layer="91"/>
 <wire x1="10.16" y1="-12.7" x2="0" y2="-12.7" width="0.1524" layer="91"/>
-</segment>
-</net>
-<net name="N$23" class="0">
+<label x="10.16" y="-10.16" size="1.778" layer="95" rot="R90"/>
+</segment>
+</net>
+<net name="USART2_RX" class="0">
 <segment>
 <pinref part="U1" gate="G$1" pin="PA3"/>
@@
 <pinref part="USART2" gate="J1" pin="1"/>
 <wire x1="33.02" y1="-15.24" x2="0" y2="-15.24" width="0.1524" layer="91"/>
+<label x="20.32" y="-15.24" size="1.778" layer="95" rot="R180"/>
 </segment>
 </net>
@@
 </segment>
 </net>
-<net name="N$17" class="0">
+<net name="SPI1_SCK" class="0">
 <segment>
 <pinref part="U1" gate="G$1" pin="PA5"/>
@@
 <pinref part="SPI1" gate="J1" pin="2"/>
 <wire x1="35.56" y1="-43.18" x2="35.56" y2="-48.26" width="0.1524" layer="91"/>
-</segment>
-</net>
-<net name="N$18" class="0">
+<label x="43.18" y="-30.48" size="1.778" layer="95" rot="R90"/>
+</segment>
+</net>
+<net name="SPI1_MISO" class="0">
 <segment>
 <pinref part="U1" gate="G$1" pin="PA6"/>
@@
 <pinref part="SPI1" gate="J1" pin="1"/>
 <wire x1="38.1" y1="-45.72" x2="38.1" y2="-48.26" width="0.1524" layer="91"/>
-</segment>
-</net>
+<label x="45.72" y="-30.48" size="1.778" layer="95" rot="R90"/>
+</segment>
+</net>

Commit message: Iteration 2 commit
Parts:
- added J2: (no value), SparkFun-Connectors:CONN_05LOCK
- added J4: (no value), SparkFun-Connectors:CONN_02
Connections:
- new net DFSDM1_CKOUT: J2.4, U1.PC2
- new net DFSDM1_DATIN0: J2.2, U1.PB1
- new net GPIO_CS: J4.1, U1.PB0
- new net SPI1_MOSI: J4.2, U1.PA7
- net 3V3: now also J2.3
- net GND: now also DAC4.2, J2.1, J2.5
Other:
- moved on the sheet: D1, D2, DAC4, R1, R2, SPI1, USART3
